Commit message: made some edition to ensure the mir250 accept the prefix /mir as it is needed when merging it with the ue

File: src/mir250_robot_ros2/mir_description/urdf/mir.urdf.xacro (robot description, xacro)
@@ -5,13 +5,14 @@
   <xacro:include filename="$(find mir_description)/urdf/include/mir_250_v1.urdf.xacro" />
   <xacro:arg name="tf_prefix" default="" />
+  <xacro:arg name="ns" default="" />
   <!-- prefix can not start with a slash like a global namespace! results in TF errors -->
-  <xacro:property name="ns" value="$(arg tf_prefix)" />
-  <xacro:if value="${ns == ''}">
+  <xacro:property name="tf_prefix_val" value="$(arg tf_prefix)" />
+  <xacro:if value="${tf_prefix_val == ''}">
     <xacro:property name="prefix" value="" />
   </xacro:if>
-  <xacro:unless value="${ns == ''}">
-    <xacro:property name="prefix" value="${ns}/" />
+  <xacro:unless value="${tf_prefix_val == ''}">
+    <xacro:property name="prefix" value="${tf_prefix_val}/" />
   </xacro:unless>
-  <xacro:mir_250 prefix="${prefix}" ns="${ns}"/>
+  <xacro:mir_250 prefix="${prefix}" ns="$(arg ns)"/>
   <!-- <xacro:diff_controller_plugin_gazebo prefix="${prefix}" ns="${ns}"
     left_wheel_joint="${prefix}left_wheel_joint"
@@ -26,5 +27,5 @@
       <plugin>gazebo_ros2_control/GazeboSystem</plugin>
     </hardware>
-    <joint name="left_wheel_joint">
+    <joint name="${prefix}left_wheel_joint">
       <command_interface name="velocity">
         <param name="min">-1</param>
@@ -34,5 +35,5 @@
       <state_interface name="velocity"/>
     </joint>
-    <joint name="right_wheel_joint">
+    <joint name="${prefix}right_wheel_joint">
       <command_interface name="velocity">
         <param name="min">-1</param>
@@ -42,33 +43,33 @@
       <state_interface name="velocity"/>
     </joint>
-    <joint name="fl_caster_rotation_joint">
+    <joint name="${prefix}fl_caster_rotation_joint">
       <state_interface name="position"/>
       <state_interface name="velocity"/>
     </joint>
-    <joint name="fr_caster_rotation_joint">
+    <joint name="${prefix}fr_caster_rotation_joint">
       <state_interface name="position"/>
       <state_interface name="velocity"/>
     </joint>
-    <joint name="bl_caster_rotation_joint">
+    <joint name="${prefix}bl_caster_rotation_joint">
       <state_interface name="position"/>
       <state_interface name="velocity"/>
     </joint>
-    <joint name="br_caster_rotation_joint">
+    <joint name="${prefix}br_caster_rotation_joint">
       <state_interface name="position"/>
       <state_interface name="velocity"/>
     </joint>
-    <joint name="fl_caster_wheel_joint">
+    <joint name="${prefix}fl_caster_wheel_joint">
       <state_interface name="position"/>
       <state_interface name="velocity"/>
     </joint>
-    <joint name="fr_caster_wheel_joint">
+    <joint name="${prefix}fr_caster_wheel_joint">
       <state_interface name="position"/>
       <state_interface name="velocity"/>
     </joint>
-    <joint name="bl_caster_wheel_joint">
+    <joint name="${prefix}bl_caster_wheel_joint">
       <state_interface name="position"/>
       <state_interface name="velocity"/>
     </joint>
-    <joint name="br_caster_wheel_joint">
+    <joint name="${prefix}br_caster_wheel_joint">
       <state_interface name="position"/>
       <state_interface name="velocity"/>

Commit message: this draft contain duplicated files after creating new merged package, saved temporarily

File: src/mir250_robot_ros2/mir_description/urdf/mir.urdf.xacro (robot description, xacro)
@@ -4,5 +4,5 @@
   <!-- MiR250 base -->
   <xacro:include filename="$(find mir_description)/urdf/include/mir_250_v1.urdf.xacro" />
-  <xacro:arg name="tf_prefix" default="" />
+  <xacro:arg name="tf_prefix" default="mir" />
   <xacro:arg name="ns" default="" />
   <!-- prefix can not start with a slash like a global namespace! results in TF errors -->

File: src/ue/Universal_Robots_ROS2_Description/urdf/ur.urdf.xacro (robot description, xacro)
@@ -1,13 +1,13 @@
 <?xml version="1.0"?>
-<robot xmlns:xacro="http://wiki.ros.org/xacro" name="$(arg name)">
+<robot xmlns:xacro="http://wiki.ros.org/xacro" name="ur">
    <!-- robot name parameter -->
-   <xacro:arg name="name" default="ur"/>
    <!-- import main macro -->
    <xacro:include filename="$(find ur_description)/urdf/ur_macro.xacro"/>
+   <xacro:arg name="name" default="ur"/>
    <!-- possible 'ur_type' values: ur3, ur5, ur10, ur3e, ur5e, ur7e, ur10e, ur12e, ur16e, ur8long, ur15, ur18, ur20, ur30 -->
    <!-- the default value should raise an error in case this was called without defining the type -->
-   <xacro:arg name="ur_type" default="ur5x"/>
+   <xacro:arg name="ur_type" default="ur5e"/>
    <!-- parameters -->
-   <xacro:arg name="tf_prefix" default="" />
+   <xacro:arg name="ur_tf_prefix" default="ur_" />
    <xacro:arg name="joint_limit_params" default="$(find ur_description)/config/$(arg ur_type)/joint_limits.yaml"/>
    <xacro:arg name="kinematics_params" default="$(find ur_description)/config/$(arg ur_type)/default_kinematics.yaml"/>
@@ -42,7 +42,7 @@
    <xacro:arg name="use_fake_hardware" default="false" />
    <xacro:arg name="fake_sensor_commands" default="false" />
-   <xacro:arg name="sim_gazebo" default="false" />
+   <xacro:arg name="sim_gazebo" default="true" />
    <xacro:arg name="sim_ignition" default="false" />
-   <xacro:arg name="simulation_controllers" default="" />
+   <xacro:arg name="simulation_controllers" default="$(find ur_simulation_gazebo)/config/ur_controllers.yaml" />
    <!-- initial position for simulations (Fake Hardware, Gazebo, Ignition) -->
    <xacro:arg name="initial_positions_file" default="$(find ur_description)/config/initial_positions.yaml"/>
@@ -58,5 +58,5 @@
          <origin rpy="0 0 0" xyz="0 0 0"/>
          <geometry>
-           <box size="5 5 0"/>
+           <box size="5 5 0.01"/>
          </geometry>
          <material name="ground_white">
@@ -80,5 +80,5 @@
    <xacro:ur_robot
      name="$(arg name)"
-     tf_prefix="$(arg tf_prefix)"
+     tf_prefix="$(arg ur_tf_prefix)"
      parent="world"
      joint_limits_parameters_file="$(arg joint_limit_params)"
@@ -134,5 +134,5 @@
       <plugin filename="libign_ros2_control-system.so" name="ign_ros2_control::IgnitionROS2ControlPlugin">
         <parameters>$(arg simulation_controllers)</parameters>
-        <controller_manager_node_name>$(arg tf_prefix)controller_manager</controller_manager_node_name>
+        <controller_manager_node_name>$(arg ur_tf_prefix)controller_manager</controller_manager_node_name>
       </plugin>
     </gazebo>
