Commit message: Modify arm position and remove Voxel layer from global map

File: src/merged/urdf/mir_ur.urdf.xacro (robot description, xacro)
@@ -117,5 +117,5 @@
     trajectory_port="$(arg trajectory_port)"
     >
-    <origin xyz="0 0 0" rpy="0 0 0" />
+    <origin xyz="0.25 0 0" rpy="0 0 0" />
   </xacro:ur_robot>
   <!-- ================================================================
